Commit message: Now with a target

File: chair_ws/src/chair/urdf/airchair.urdf.xacro (robot description, xacro)
@@ -4,4 +4,5 @@
         modelled after the wheelchair
         This robot has a camera
+        It now has a target
 	Version 1.0.
 	-->
@@ -20,5 +21,5 @@
   <xacro:property name="robot_caster_link_length" value="0.03" />
   <xacro:property name="robot_caster_link_offset" value="-0.025" />
-  <xacro:property name="robot_caster_joint_offset" value="${robot_base_length/2-0.01}" />
+  <xacro:property name="robot_caster_joint_offset" value="${robot_base_length/2}" />
   <xacro:property name="robot_caster_wheel_radius" value="0.098" />
   <xacro:property name="robot_caster_wheel_width" value="0.02" />
@@ -28,4 +29,9 @@
   <xacro:property name="robot_camera_xoffset" value="-0.4" />
   <xacro:property name="robot_camera_zoffset" value="1.1" />
+  <xacro:property name="target_width" value="0.45" />
+  <xacro:property name="target_length" value="0.01" />
+  <xacro:property name="target_height" value="0.60" />
+  <xacro:property name="target_xoffset" value="-0.45" />
+  <xacro:property name="target_zoffset" value="-0.3" />
   <!-- Import colors defined externally -->
   <xacro:include filename="$(find chair)/colors.xacro" />
@@ -68,4 +74,28 @@
     <parent link="base_footprint" />
     <child link="base_link" />
+    <axis xyz="0 0 1" />
+  </joint>
+  <!-- Visual Target -->
+  <gazebo reference="target_link">
+    <material>apriltag_36h10</material>
+  </gazebo>
+  <link name="target_link">
+    <visual>
+      <geometry>
+        <box size="${target_length} ${target_width} ${target_height}" />
+      </geometry>
+      <material name="green"/>
+    </visual>
+    <collision>
+      <geometry>
+        <box size="${target_length} ${target_width} ${target_height}" />
+      </geometry>
+    </collision>
+    <xacro:I_cuboid m="0.01" x="${target_length}" y="${target_width}" z="${target_height}" />
+  </link>
+  <joint name="target_joint" type="fixed">
+    <origin xyz="${target_xoffset} 0.0 ${target_zoffset+target_height/2}" rpy="0.0 0.0 0.0" />
+    <parent link="base_link" />
+    <child link="target_link" />
     <axis xyz="0 0 1" />
   </joint>
@@ -202,5 +232,5 @@
     <parent link="base_link" />
     <child link="left_caster_link" />
-    <origin rpy="0 0 3.1415" xyz="${robot_caster_joint_offset-robot_caster_link_width/2} ${robot_base_width/2-robot_caster_link_length/2} ${-robot_base_height/2-robot_caster_link_height/2}" />
+    <origin rpy="0 0 3.1415" xyz="${robot_caster_joint_offset-robot_caster_link_width/2} ${robot_base_width/2-robot_caster_link_length/2-0.015} ${-robot_base_height/2-robot_caster_link_height/2}" />
   </joint>
   <joint name="right_caster_joint" type="continuous">
@@ -208,5 +238,5 @@
     <parent link="base_link" />
     <child link="right_caster_link" />
-    <origin rpy="0 0 3.1415" xyz="${robot_caster_joint_offset-robot_caster_link_width/2} ${-robot_base_width/2+robot_caster_link_length/2} ${-robot_base_height/2-robot_caster_link_height/2}" />
+    <origin rpy="0 0 3.1415" xyz="${robot_caster_joint_offset-robot_caster_link_width/2} ${-robot_base_width/2+robot_caster_link_length/2+0.015} ${-robot_base_height/2-robot_caster_link_height/2}" />
   </joint>
   <!-- caster wheel -->

Commit message: multiple chairs working

File: chair_ws/src/chair/urdf/airchair.urdf.xacro (robot description, xacro)
@@ -9,4 +9,8 @@
 <robot name="$(arg name)" xmlns:xacro="http://www.ros.org/wiki/xacro">
   <!-- Define the robot -->
+  <xacro:arg name="robot_name" default="chair" />
+  <xacro:property name="robot_name" value="$(arg name)" />
+  <xacro:arg name="target" default="apriltag_36h10_0" />
+  <xacro:property name="target" value="$(arg target)" />
   <xacro:property name="robot_base_width" value="0.556" />
   <xacro:property name="robot_base_length" value="0.504" />
@@ -140,5 +144,8 @@
       </camera>
       <plugin name="camera_controller" filename="libgazebo_ros_camera.so">
-        <camera_name>mycamera</camera_name>
+        <ros>
+          <namespace>/${robot_name}</namespace>
+        </ros>
+        <camera_name>camera</camera_name>
         <frame_name>camera_link</frame_name>
       </plugin>
@@ -289,4 +296,7 @@
   <gazebo>
     <plugin name="joint_state_publisher" filename="libgazebo_ros_joint_state_publisher.so">
+      <ros>
+        <namespace>/${robot_name}</namespace>
+      </ros>
       <update_rate>100</update_rate>
       <joint_name>left_caster_wheel_joint</joint_name>
@@ -299,4 +309,7 @@
   <gazebo>
     <plugin name="differential_drive_controller" filename="libgazebo_ros_diff_drive.so">
+      <ros>
+        <namespace>/${robot_name}</namespace>
+      </ros>
       <update_rate>20</update_rate>
       <left_joint>left_wheel_joint</left_joint>

Commit message: fixed bug in urdf

File: chair_ws/src/chair/urdf/airchair.urdf.xacro (robot description, xacro)
@@ -82,5 +82,5 @@
   <!-- Visual Target -->
   <gazebo reference="target_link">
-    <material>apriltag_36h10</material>
+    <material>${target}</material>
   </gazebo>
   <link name="target_link">

Commit message: lower resolution model for performance

File: chair_ws/src/chair/urdf/airchair.urdf.xacro (robot description, xacro)
@@ -9,4 +9,6 @@
 <robot name="$(arg name)" xmlns:xacro="http://www.ros.org/wiki/xacro">
   <!-- Define the robot -->
+  <xacro:arg name="show_video" default="true" />
+  <xacro:property name="show_video" value="$(arg show_video)" />
   <xacro:arg name="robot_name" default="chair" />
   <xacro:property name="robot_name" value="$(arg name)" />
@@ -130,5 +132,5 @@
   <gazebo reference="camera_link">
     <sensor type="camera" name="camera">
-      <visualize>true</visualize>
+      <visualize>${show_video}</visualize>
       <camera>
         <horizontal_fov>${65 * 3.1415/180}</horizontal_fov>
@@ -155,8 +157,8 @@
   <link name="left_wheel_link">
     <visual>
-      <origin rpy="0 1.5708 0" xyz="0 0 0" />
-      <geometry>
-        <!--cylinder length="${robot_wheel_width}" radius="${robot_wheel_radius}" -->
-        <mesh filename="$(find chair)/rearwheel.obj" scale="0.001 0.001 0.001"/>
+      <!-- origin rpy="0 1.5708 0" xyz="0 0 0" -->
+      <geometry>
+        <cylinder length="${robot_wheel_width}" radius="${robot_wheel_radius}" />
+        <!-- mesh filename="$(find chair)/rearwheel.obj" scale="0.001 0.001 0.001"-->>
       </geometry>
     </visual>
@@ -177,8 +179,8 @@
   <link name="right_wheel">
     <visual>
-      <origin rpy="0 1.5708 0" xyz="0 0 0" />
-      <geometry>
-        <!-- cylinder length="${robot_wheel_width}" radius="${robot_wheel_radius}" -->
-        <mesh filename="$(find chair)/rearwheel.obj" scale="0.001 0.001 0.001"/>
+      <!-- origin rpy="0 1.5708 0" xyz="0 0 0" -->
+      <geometry>
+        <cylinder length="${robot_wheel_width}" radius="${robot_wheel_radius}" />
+        <!-- mesh filename="$(find chair)/rearwheel.obj" scale="0.001 0.001 0.001"-->
       </geometry>
     </visual>

Commit message: tilted camera

File: chair_ws/src/chair/urdf/airchair.urdf.xacro (robot description, xacro)
@@ -5,8 +5,11 @@
         This robot has a camera
         It now has a target
-	Version 1.0.
+        It now tilts the camera
+	Version 1.2.
 	-->
 <robot name="$(arg name)" xmlns:xacro="http://www.ros.org/wiki/xacro">
   <!-- Define the robot -->
+  <xacro:arg name="camera_tilt" default="0.0" />
+  <xacro:property name="camera_tilt" value="$(arg camera_tilt)" />
   <xacro:arg name="show_video" default="true" />
   <xacro:property name="show_video" value="$(arg show_video)" />
@@ -125,5 +128,5 @@
   </link>
   <joint name="camera_joint" type="fixed">
-    <origin xyz="${robot_camera_xoffset} 0.0 ${robot_camera_zoffset+robot_camera_height/2}" rpy="0.0 0.0 0.0" />
+    <origin xyz="${robot_camera_xoffset} 0.0 ${robot_camera_zoffset+robot_camera_height/2}" rpy="0 ${camera_tilt} 0" />
     <parent link="base_link" />
     <child link="camera_link" />
